File: pcb/v1.0-uni/smallcat-uni.kicad_pcb (KiCad board)
At the start: 2 copper layers, 199.7 x 97.2 mm, 28 parts, among them SW10 SW_Push, SW11 SW_Push, SW11_r1 SW_Push, SW12 SW_Push, SW12_r1 SW_Push, SW15 SW_Push, SW15_r1 SW_Push, SW16 SW_Push, SW17 SW_Push, SW18_r1 SW_Push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

Commit message: Edit README
Other:
- board text added: "place me face up (components showing)"
